File: Clone_Board/Clone_Board_PCB_Files/Clone Board.kicad_sch (KiCad schematic)
At the start: 14 parts, among them SW1 SW_SPDT, U1 STM32F401CEUx

Commit message: Updated log and PCB files
Parts:
- removed SW1: SW_SPDT, symbol Switch:SW_SPDT
- added C11: 0.1uF, Capacitor_SMD:C_0805_2012Metric_Pad1.18x1.45mm_HandSolder, symbol Device:C
- added C12: 10uF, Capacitor_SMD:C_0805_2012Metric_Pad1.18x1.45mm_HandSolder, symbol Device:C
- added J1: USB_C_Receptacle_USB2.0_16P, Connector_USB:USB_C_Receptacle_GCT_USB4105-xx-A_16P_TopMnt_Horizontal, symbol Connector:USB_C_Receptacle_USB2.0_16P
- added R3, R4: 5.1kOhm, Resistor_SMD:R_0805_2012Metric_Pad1.20x1.40mm_HandSolder, symbol Device:R
- added SW1, SW2: SW_Push, Button_Switch_SMD:SW_Push_1P1T_NO_CK_KSC6xxJ, symbol Switch:SW_Push
Connections:
- net +3.3V: now also R2.1, SW1.1; no longer R2.2
- net Boot0: now also R1.2, SW1.2
- net GND: now also C11.1, C12.1, J1.A1 (GND), J1.A12 (GND), J1.B1 (GND), J1.B12 (GND), J1.SH (SHIELD), R3.2, R4.2, SW2.2
- net NRST: now reaches U1.7 (NRST)
- net NRST: now also R2.2, C11.2, SW2.1; no longer R2.1
- net USB_DM: now reaches U1.32 (PA11)
- net USB_DM: now also J1.A7 (D-), J1.B7 (D-)
- net USB_DP: now reaches U1.33 (PA12)
- net USB_DP: now also J1.A6 (D+), J1.B6 (D+)
- new net: J1.A5 (CC1), R3.1
- new net: C12.2, J1.A4 (VBUS), J1.A9 (VBUS), J1.B4 (VBUS), J1.B9 (VBUS)
- new net: J1.B5 (CC2), R4.1
- no-connect marks 0 -> 2
Other:
- note added: "Boot0 and NRST Pin Protection"
- note added: "Chip Power Scheme"
- moved on the sheet: C10, C2, C3, C4, C5, C6, C7, C8, C9, R1
